File: kicad/MicroXTSD.kicad_sch (KiCad schematic)
At the start: 25 parts, among them J2 SD_Adapter, J3 IRQ, U1 HCT245, U10 AHCT138, U11 28C64, U2 HCT573, U3 HCT573, U4 HCT245, U5 HCT04, U6 HCT32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

Commit message: Revision 3
Connections:
- net GND: now also U6.10
- net VCC: no longer U6.10
Changed lines of the file:
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@@
     (pin "2")
-  )
-  (symbol (lib_id "power:VCC") (at 31.75 161.29 90) (unit 1)
-    (in_bom yes) (on_board yes)
-    (property "Reference" "#PWR0106" (id 0) (at 35.56 161.29 0)
-      (effects (font (size 1.27 1.27)) hide)
-    )
-    (property "Value" "VCC" (id 1) (at 29.21 161.29 90)
-      (effects (font (size 1.27 1.27)) (justify left))
-    )
-    (property "Footprint" "" (id 2) (at 31.75 161.29 0)
-      (effects (font (size 1.27 1.27)) hide)
-    )
-    (property "Datasheet" "" (id 3) (at 31.75 161.29 0)
-      (effects (font (size 1.27 1.27)) hide)
-    )
-    (pin "1")
   )
   (symbol (lib_id "Micro-XTCF-rescue:GND-xt-cf-rescue-xt-cf-mini-rescue") (at 90.805 252.095 0) (unit 1)
@@
     )
     (property "Datasheet" "" (id 3) (at 137.16 221.615 0)
+      (effects (font (size 1.27 1.27)) hide)
+    )
+    (pin "1")
+  )
+  (symbol (lib_id "power:GND") (at 31.75 161.29 270) (unit 1)
+    (in_bom yes) (on_board yes)
+    (property "Reference" "#PWR?" (id 0) (at 25.4 161.29 0)
+      (effects (font (size 1.27 1.27)) hide)
+    )
+    (property "Value" "GND" (id 1) (at 28.4988 161.417 90)
+      (effects (font (size 1.27 1.27)) (justify right))
+    )
+    (property "Footprint" "" (id 2) (at 31.75 161.29 0)
+      (effects (font (size 1.27 1.27)) hide)
+    )
+    (property "Datasheet" "" (id 3) (at 31.75 161.29 0)
       (effects (font (size 1.27 1.27)) hide)
     )
@@
       (reference "#PWR0105") (unit 1) (value "GND") (footprint "")
     )
-    (path "/02567d70-58ef-4d85-b16e-7663601b34ce"
-      (reference "#PWR0106") (unit 1) (value "VCC") (footprint "")
-    )
     (path "/d58aa45d-7be5-4bd1-8ddc-c8ce52c2e8c6"
       (reference "#PWR0107") (unit 1) (value "VCC") (footprint "")
@@
       (reference "#PWR0110") (unit 1) (value "GND") (footprint "")
     )
+    (path "/5f28dc32-7ee6-42e1-80b3-d8428e7a8471"
+      (reference "#PWR?") (unit 1) (value "GND") (footprint "")
+    )
     (path "/00000000-0000-0000-0000-00005dd75d44"
